File: Schematics/DSKY.brd (EAGLE design)
At the start: 100 x 80 mm, 6 parts, among them IC1 74LS595N, IC2 74LS595N, IC3 74LS595N

Commit message: Update shit
Parts:
- moved IC2 35.8 mm to (20.3, 69.8)
- moved IC1 14.5 mm to (47.0, 69.8)
- moved SV1 8.89 mm to (5.08, 49.5)
- moved IC3 4.02 mm to (76.2, 69.8)
- moved U$1 2.54 mm to (26.7, 16.5)
- moved D2 1.80 mm to (68.6, 14.0)
Routing:
- net N$15: track 222.9 -> 107.3 mm, vias 1 -> 0
- net N$25: track 77.6 -> 36.2 mm, vias 2 -> 0
- net N$1: track 99.0 -> 58.6 mm
- net N$7: track 97.8 -> 65.2 mm, vias 4 -> 0
- net N$26: track 28.2 -> 0.00 mm, vias 1 -> 0
- net N$12: track 93.4 -> 67.1 mm, vias 1 -> 0
- net N$5: track 86.8 -> 63.1 mm, vias 3 -> 0
- net N$20: track 39.2 -> 15.5 mm, vias 1 -> 0
- net N$21: track 39.7 -> 17.9 mm, vias 1 -> 0
- net N$3: track 91.7 -> 75.7 mm, vias 8 -> 0
- net N$6: track 64.3 -> 52.9 mm
- net N$14: track 60.3 -> 49.8 mm, vias 2 -> 0
- net N$13: track 62.3 -> 51.8 mm, vias 4 -> 0
- net N$4: track 79.4 -> 69.1 mm, vias 4 -> 0
- net N$18: track 100.1 -> 91.2 mm
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